File: 64MB-SIMM/64MB-SIMM.kicad_sch (KiCad schematic)
At the start: 1 part

Commit message: Updated 64 SIMM for release
Parts:
- removed J?: SIMM, symbol CPS3:SIMM
- added C1: 100uf, Capacitor_Tantalum_SMD:CP_EIA-3528-12_Kemet-T, symbol Device:C_Polarized_Small_US
- added C10, C11, C12, C13, C14, C15, C16, C17, C18, C4, C5, C6, C7, C8, C9: 100nf, Capacitor_SMD:C_0603_1608Metric, symbol Device:C_Small
- added C2, C3: 10uf, Capacitor_Tantalum_SMD:CP_EIA-3216-10_Kemet-I, symbol Device:C_Polarized_Small_US
- added J1: 64MB, CPS3:SIMM_EDGE, symbol 5822030-3:5822030-3
- added J2: Conn_02x03_Odd_Even, Connector_PinSocket_1.27mm:PinSocket_2x03_P1.27mm_Horizontal, symbol Connector_Generic:Conn_02x03_Odd_Even
- added R1, R2, R3, R4: 10K, Resistor_SMD:R_0603_1608Metric, symbol Device:R_US
- added U1: LM1117-3.3, Package_TO_SOT_SMD:SOT-223-3_TabPin2, symbol Regulator_Linear:AMS1117-3.3
- added U10, U4: S29GL256/512/01G, Package_SO:TSOP-I-56_18.4x14mm_P0.5mm, symbol CPS3:29GL128
- added U2, U3, U7, U9: 74LVC4245A, Package_SO:TSSOP-24_4.4x7.8mm_P0.65mm, symbol Logic_LevelTranslator:SN74LVC8T245
- added U5, U6: 74LVC245A, Package_SO:TSSOP-20_4.4x6.5mm_P0.65mm, symbol Logic_LevelTranslator:SN74LVC245APW
- added U8: 74LVC827, Package_SO:TSSOP-24_4.4x7.8mm_P0.65mm, symbol 74xx:74LVC827
Connections:
- net A0: now also U10.31 (A0), U4.31 (A0), U8.14 (Y10)
- net A1: now also U10.26 (A1), U4.26 (A1), U8.17 (Y7)
- net A10: now also U10.8 (A10), U4.8 (A10), U5.12 (B7)
- net A11: now also U10.7 (A11), U4.7 (A11), U5.13 (B6)
- net A12: now also U10.6 (A12), U4.6 (A12), U5.18 (B1)
- net A13: now also U10.5 (A13), U4.5 (A13), U5.17 (B2)
- net A14: now also U10.4 (A14), U4.4 (A14), U5.16 (B3)
- net A15: now also U10.3 (A15), U4.3 (A15), U5.15 (B4)
- net A16: now also U10.54 (A16), U4.54 (A16), U5.14 (B5)
- net A17: now also U10.19 (A17), U4.19 (A17), U6.11 (B8)
- net A18: now also U10.18 (A18), U4.18 (A18), U6.12 (B7)
- net A19: now also U10.11 (A19), U4.11 (A19), U6.17 (B2)
- net A2: now also U10.25 (A2), U4.25 (A2), U8.18 (Y6)
- net A20: now also U10.12 (A20), U4.12 (A20), U6.16 (B3)
- net A3: now also U10.24 (A3), U4.24 (A3), U8.19 (Y5)
- net A4: now also U10.23 (A4), U4.23 (A4), U8.20 (Y4)
- net A5: now also U10.22 (A5), U4.22 (A5), U8.21 (Y3)
- net A6: now also U10.21 (A6), U4.21 (A6), U8.22 (Y2)
- net A7: now also U10.20 (A7), U4.20 (A7), U8.23 (Y1)
- net A8: now also U10.10 (A8), U4.10 (A8), U6.18 (B1)
- net A9: now also U10.9 (A9), U4.9 (A9), U5.11 (B8)
- net CE: now also U10.32 (CE), U4.32 (CE), U8.15 (Y9)
- net GND: now also C1.2, C10.2, C11.2, C12.2, C13.2, C14.2, C15.2, C16.2, C17.2, C18.2, C2.2, C3.2, C4.2, C5.2, C6.2, C7.2, C8.2, C9.2, J1.11, J1.20, J1.29, J1.49, J1.61, J1.63, J1.68, J2.6 (Pin_6), U1.1 (GND), U10.33 (GND), U10.52 (GND), U10.55 (A25), U10.56 (A24), U2.11 (GND), U2.12 (GND), U2.13 (GND), U3.11 (GND), U3.12 (GND), U3.13 (GND), U4.33 (GND), U4.52 (GND), U4.55 (A25), U4.56 (A24), U5.10 (GND), U5.19 (~{OE}), U6.10 (GND), U6.19 (~{OE}), U7.11 (GND), U7.12 (GND), U7.13 (GND), U8.1 (~{OE1}), U8.12 (GND), U8.13 (~{OE2}), U9.11 (GND), U9.12 (GND), U9.13 (GND)
- net OE: now also U10.34 (OE), U4.34 (OE), U8.16 (Y8)
- net RST: now also U10.14 (RESET), U4.14 (RESET), U6.13 (B6)
- net VCC: now also C1.1, C13.1, C14.1, C2.1, C4.1, C6.1, J1.1, J1.2, R4.1, U1.3 (VI), U2.1 (V_{CCA}), U3.1 (V_{CCA}), U7.1 (V_{CCA}), U9.1 (V_{CCA})
- new net A21: J2.1 (Pin_1), J2.2 (Pin_2), R1.2, U10.15 (A21), U4.15 (A21)
- new net A22: J2.3 (Pin_3), J2.4 (Pin_4), R2.2, U10.2 (A22), U4.2 (A22)
- new net A23: J2.5 (Pin_5), R3.2, U10.1 (A23), U4.1 (A23)
- new net SA0: J1.60, U8.11 (A10)
- new net SA1: J1.59, U8.8 (A7)
- new net SA10: J1.50, U5.8 (A7)
- new net SA11: J1.48, U5.7 (A6)
- new net SA12: J1.47, U5.2 (A1)
- new net SA13: J1.46, U5.3 (A2)
- new net SA14: J1.45, U5.4 (A3)
- new net SA15: J1.44, U5.5 (A4)
- new net SA16: J1.43, U5.6 (A5)
- new net SA17: J1.42, U6.9 (A8)
- new net SA18: J1.41, U6.8 (A7)
- new net SA19: J1.40, U6.3 (A2)
- new net SA2: J1.58, U8.7 (A6)
- new net SA20: J1.39, U6.4 (A3)
- new net SA3: J1.57, U8.6 (A5)
- new net SA4: J1.56, U8.5 (A4)
- new net SA5: J1.55, U8.4 (A3)
- new net SA6: J1.54, U8.3 (A2)
- new net SA7: J1.53, U8.2 (A1)
- new net SA8: J1.52, U6.2 (A1)
- new net SA9: J1.51, U5.9 (A8)
- new net SCE: J1.67, R4.2, U2.22 (~{OE}), U3.22 (~{OE}), U7.22 (~{OE}), U8.10 (A9), U9.22 (~{OE})
- new net SHD0: U10.35 (D0), U9.21 (B1)
- new net SHD1: U10.37 (D1), U9.19 (B3)
- new net SHD10: U10.40 (D10), U9.16 (B6)
- new net SHD11: U10.42 (D11), U9.14 (B8)
- new net SHD12: U10.45 (D12), U7.20 (B2)
- new net SHD13: U10.47 (D13), U7.18 (B4)
- new net SHD14: U10.49 (D14), U7.16 (B6)
- new net SHD15: U10.51 (A-1/D15), U7.14 (B8)
- new net SHD2: U10.39 (D2), U9.17 (B5)
- new net SHD3: U10.41 (D3), U9.15 (B7)
- new net SHD4: U10.44 (D4), U7.21 (B1)
- new net SHD5: U10.46 (D5), U7.19 (B3)
- new net SHD6: U10.48 (D6), U7.17 (B5)
- new net SHD7: U10.50 (D7), U7.15 (B7)
- new net SHD8: U10.36 (D8), U9.20 (B2)
- new net SHD9: U10.38 (D9), U9.18 (B4)
- new net SND_AD0: U3.21 (B1), U4.35 (D0)
- new net SND_AD1: U3.19 (B3), U4.37 (D1)
- new net SND_AD10: U3.16 (B6), U4.40 (D10)
- new net SND_AD11: U3.14 (B8), U4.42 (D11)
- new net SND_AD12: U2.20 (B2), U4.45 (D12)
- new net SND_AD13: U2.18 (B4), U4.47 (D13)
- new net SND_AD14: U2.16 (B6), U4.49 (D14)
- new net SND_AD15: U2.14 (B8), U4.51 (A-1/D15)
- new net SND_AD2: U3.17 (B5), U4.39 (D2)
- new net SND_AD3: U3.15 (B7), U4.41 (D3)
- new net SND_AD4: U2.21 (B1), U4.44 (D4)
- new net SND_AD5: U2.19 (B3), U4.46 (D5)
- new net SND_AD6: U2.17 (B5), U4.48 (D6)
- new net SND_AD7: U2.15 (B7), U4.50 (D7)
- new net SND_AD8: U3.20 (B2), U4.36 (D8)
- new net SND_AD9: U3.18 (B4), U4.38 (D9)
- new net SOE: J1.71, U2.2 (DIR), U3.2 (DIR), U7.2 (DIR), U8.9 (A8), U9.2 (DIR)
- new net SRST: J1.62, U6.7 (A6)
- new net SSHD0: J1.28, U9.3 (A1)
- new net SSHD1: J1.27, U9.5 (A3)
- new net SSHD10: J1.35, U9.8 (A6)
- new net SSHD11: J1.34, U9.10 (A8)
- new net SSHD12: J1.33, U7.4 (A2)
- new net SSHD13: J1.32, U7.6 (A4)
- new net SSHD14: J1.31, U7.8 (A6)
- new net SSHD15: J1.30, U7.10 (A8)
- new net SSHD2: J1.26, U9.7 (A5)
- new net SSHD3: J1.25, U9.9 (A7)
- new net SSHD4: J1.24, U7.3 (A1)
- new net SSHD5: J1.23, U7.5 (A3)
- new net SSHD6: J1.22, U7.7 (A5)
- new net SSHD7: J1.21, U7.9 (A7)
- new net SSHD8: J1.37, U9.4 (A2)
- new net SSHD9: J1.36, U9.6 (A4)
- new net SSND_AD0: J1.10, U3.3 (A1)
- new net SSND_AD1: J1.9, U3.5 (A3)
- new net SSND_AD10: J1.17, U3.8 (A6)
- new net SSND_AD11: J1.16, U3.10 (A8)
- new net SSND_AD12: J1.15, U2.4 (A2)
- new net SSND_AD13: J1.14, U2.6 (A4)
- new net SSND_AD14: J1.13, U2.8 (A6)
- new net SSND_AD15: J1.12, U2.10 (A8)
- new net SSND_AD2: J1.8, U3.7 (A5)
- new net SSND_AD3: J1.7, U3.9 (A7)
- new net SSND_AD4: J1.6, U2.3 (A1)
- new net SSND_AD5: J1.5, U2.5 (A3)
- new net SSND_AD6: J1.4, U2.7 (A5)
- new net SSND_AD7: J1.3, U2.9 (A7)
- new net SSND_AD8: J1.19, U3.4 (A2)
- new net SSND_AD9: J1.18, U3.6 (A4)
- new net SWE_SH: J1.69, U6.6 (A5)
- new net SWE_SND: J1.70, U6.5 (A4)
- new net VDD: C10.1, C11.1, C12.1, C15.1, C16.1, C17.1, C18.1, C3.1, C5.1, C7.1, C8.1, C9.1, R1.1, R2.1, R3.1, U1.2 (VO), U10.29 (VIO), U10.43 (VCC), U10.53 (RFU/BYTE), U2.23 (V_{CCB}), U2.24 (V_{CCB}), U3.23 (V_{CCB}), U3.24 (V_{CCB}), U4.29 (VIO), U4.43 (VCC), U4.53 (RFU/BYTE), U5.1 (DIR), U5.20 (VCC), U6.1 (DIR), U6.20 (VCC), U7.23 (V_{CCB}), U7.24 (V_{CCB}), U8.24 (VCC), U9.23 (V_{CCB}), U9.24 (V_{CCB})
- new net WE_SH: U10.13 (WE), U6.14 (B5)
- new net WE_SND: U4.13 (WE), U6.15 (B4)
- no-connect marks 8 -> 11
