File: src/SIMM-SWITCH/SIMM-SWITCH.kicad_pcb (KiCad board)
At the start: 2 copper layers, 122.5 x 36.6 mm, 7 parts, among them J1 Conn_02x03_Odd_Even, J2 Conn_02x03_Odd_Even, J3 Conn_02x03_Odd_Even, J4 Conn_02x03_Odd_Even, J5 Conn_02x03_Odd_Even, J6 Conn_02x03_Odd_Even, SW1 SW_DIP_x03

Commit message: Updated footprints
Parts:
- SW1: footprint herzmx:SW-SMD_6P-L8.6-W6.2-P2.54-LS9.8 -> CPS3:SW-SMD_6P-L8.6-W6.2-P2.54-LS9.8
