File: src/SIMM-SWITCH/SIMM-SWITCH.kicad_sch (KiCad schematic)
At the start: 7 parts, among them J1 Conn_02x03_Odd_Even, J2 Conn_02x03_Odd_Even, J3 Conn_02x03_Odd_Even, J4 Conn_02x03_Odd_Even, J5 Conn_02x03_Odd_Even, J6 Conn_02x03_Odd_Even, SW1 SW_DIP_x03

Commit message: Updated footprints
Parts:
- J1, J2, J3, J4, J5, J6: LCSC (none) -> C2881908
- SW1: footprint herzmx:SW-SMD_6P-L8.6-W6.2-P2.54-LS9.8 -> CPS3:SW-SMD_6P-L8.6-W6.2-P2.54-LS9.8; LCSC (none) -> C319040
Changed lines of the file:
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@@
+			)
+		)
+		(property "LCSC" "C2881908"
+			(at 69.85 90.17 0)
+			(effects
+				(font
+					(size 1.27 1.27)
+				)
+				(hide yes)
 			)
 		)
@@
 			)
 		)
+		(property "LCSC" "C2881908"
+			(at 120.65 90.17 0)
+			(effects
+				(font
+					(size 1.27 1.27)
+				)
+				(hide yes)
+			)
+		)
 		(pin "3"
 		)
@@
 			)
 		)
+		(property "LCSC" "C2881908"
+			(at 121.92 105.41 0)
+			(effects
+				(font
+					(size 1.27 1.27)
+				)
+				(hide yes)
+			)
+		)
 		(pin "3"
 		)
@@
 			)
 		)
+		(property "LCSC" "C2881908"
+			(at 69.85 106.68 0)
+			(effects
+				(font
+					(size 1.27 1.27)
+				)
+				(hide yes)
+			)
+		)
 		(pin "3"
 		)
@@
 			)
 		)
+		(property "LCSC" "C2881908"
+			(at 96.52 106.68 0)
+			(effects
+				(font
+					(size 1.27 1.27)
+				)
+				(hide yes)
+			)
+		)
 		(pin "3"
 		)
@@
 			)
 		)
+		(property "LCSC" "C2881908"
+			(at 95.25 90.17 0)
+			(effects
+				(font
+					(size 1.27 1.27)
+				)
+				(hide yes)
+			)
+		)
 		(pin "3"
 		)
@@
 			)
 		)
-		(property "Footprint" "herzmx:SW-SMD_6P-L8.6-W6.2-P2.54-LS9.8"
+		(property "Footprint" "CPS3:SW-SMD_6P-L8.6-W6.2-P2.54-LS9.8"
 			(at 72.39 128.27 0)
 			(effects
@@
 			(at 72.39 125.73 0)
 			(effects
+				(font
+					(size 1.27 1.27)
+				)
+				(hide yes)
+			)
+		)
+		(property "LCSC" "C319040"
+			(at 72.39 125.73 0)
+			(effects
