File: src/128MB-SIMM/128MB-SIMM.kicad_pcb (KiCad board)
At the start: 4 copper layers, 108 x 25.3 mm, 35 parts, among them J2 Conn_02x03_Odd_Even, J4 128MB, U1 LM1117-3.3, U2 74LVC4245A, U3 74LVC4245A, U4 S29GL01GS, U5 74LVC245A, U6 74LVC245A, U7 74LVC245A, U8 74LVC245A, U9 74LS148

Commit message: update source files changed LS41 by LVC00 and LVC08
Parts:
- removed the C12 at (179.8, 94.4)
- removed the R4 at (190.5, 89.6)
- removed the U7 at (172.6, 96.5)
- added C14: 100nf, Capacitor_SMD:C_0603_1608Metric, F.Cu at (180.5, 85.3)
- added U8: LVC00A, Package_SO:TSSOP-14_4.4x5mm_P0.65mm, F.Cu at (184.0, 96.5)
- C12: renamed from C13; moved to F.Cu
- U9: value 74LS148 -> LVC08A; footprint Package_SO:SOIC-16_3.9x9.9mm_P1.27mm -> Package_SO:TSSOP-14_4.4x5mm_P0.65mm; moved to F.Cu
- moved U4 11.4 mm to (172.6, 96.5)
- moved U9 7.75 mm to (184.0, 87.4), turned to 90 degrees
- moved C12 5.21 mm to (180.5, 94.4), turned to -90 degrees
- turned R1 to 0 degrees
- renumbered C14 to C13, C3 to C2, C5 to C3, C2 to C4, C4 to C5, C7 to C6, C6 to C7, J4 to J1, R5 to R1, R1 to R2, R2 to R3, R3 to R4, U8 to U4, U6 to U5, U5 to U6, U4 to U7
Connections:
- C12 pad 1: VCC -> VDD
- R1 pad 1: /SCE -> /ROMCE
- R1 pad 2: VCC -> VDD
- U2 pad 22: /SCE -> /ROMCE
- U3 pad 22: /SCE -> /ROMCE
- U5 pad 11: /A8 -> /A7
- U5 pad 12: /A9 -> /A17
- U5 pad 13: /A10 -> /A18
- U5 pad 14: unconnected-(U6-B5-Pad14) -> /RST
- U5 pad 15: /ROMCE -> /WE
- U5 pad 16: unconnected-(U6-B3-Pad16) -> /A20
- U5 pad 17: /A11 -> /A19
- U5 pad 18: unconnected-(U6-B1-Pad18) -> /A8
- U5 pad 2: VDD -> /SA8
- U5 pad 3: /SA11 -> /SA19
- U5 pad 4: GND -> /SA20
- U5 pad 5: /SCE -> /SWE
- U5 pad 6: GND -> /SRST
- U5 pad 7: /SA10 -> /SA18
- U5 pad 8: /SA9 -> /SA17
- U5 pad 9: /SA8 -> /SA7
- U6 pad 11: unconnected-(U5-B8-Pad11) -> /A9
- U6 pad 12: /A16 -> /A10
- U6 pad 13: /A22 -> /A11
- U6 pad 14: /A15 -> /A16
- U6 pad 15: /A14 -> /A15
- U6 pad 16: /A13 -> /A14
- U6 pad 17: /A12 -> /A13
- U6 pad 18: unconnected-(U5-B1-Pad18) -> /A12
- U6 pad 2: VDD -> /SA12
- U6 pad 3: /SA12 -> /SA13
- U6 pad 4: /SA13 -> /SA14
- U6 pad 5: /SA14 -> /SA15
- U6 pad 6: /SA15 -> /SA16
- U6 pad 7: /SA22 -> /SA11
- U6 pad 8: /SA16 -> /SA10
- U6 pad 9: GND -> /SA9
- U9 pad 10: Net-(U9-I1) -> /CEAB
- U9 pad 11: Net-(U9-I1) -> /CEAB
- U9 pad 12: Net-(U9-I1) -> /CEB
- U9 pad 13: Net-(U9-I1) -> /CEA
- U9 pad 14: /SCE -> VDD
- U9 pad 3: /CEC -> unconnected-(U9-Pad3)
- U9 pad 4: /CED -> /CEC
- U9 pad 5: GND -> /CED
- U9 pad 6: unconnected-(U9-S2-Pad6) -> /CECD
- U9 pad 7: /SA22 -> GND
- U9 pad 8: GND -> /ROMCE
- U9 pad 9: /SA21 -> /CECD
Routing:
- net /SCE: track 96.7 -> 0.00 mm, vias 2 -> 0
- net VCC: track 145.8 -> 57.3 mm
- net /ROMCE: track 47.2 -> 99.8 mm
- net /SA22: track 51.5 -> 0.00 mm, vias 1 -> 0
- net /A22: track 13.3 -> 51.0 mm, vias 0 -> 2
- net /SA0: track 24.2 -> 4.48 mm, vias 3 -> 0
- net /SA5: track 24.1 -> 5.97 mm, vias 2 -> 0
- net /A21: track 37.3 -> 54.8 mm, vias 0 -> 2
- net Net-(U9-I1): track 15.7 -> 0.00 mm, vias 2 -> 0
- net /SA6: track 23.8 -> 10.2 mm, vias 2 -> 0
- net /SOE: track 120.2 -> 133.6 mm, vias 1 -> 2
- net /SA21: track 13.2 -> 0.00 mm, vias 3 -> 0
- net /SA7: track 17.4 -> 4.70 mm
- net GND: track 77.7 -> 65.1 mm
- net /A0: track 73.0 -> 60.4 mm
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